File: project/clockradio/_autosave-clockradio.kicad_sch (KiCad schematic)
At the start: 12 parts, among them U1 LM386

Commit message: updates to project schematic
Parts:
- added U2: RP2040, Package_DFN_QFN:QFN-56-1EP_7x7mm_P0.4mm_EP3.2x3.2mm, symbol MCU_RaspberryPi:RP2040
Connections:
- net LOUT is gone; now on net +1V0: RDA58007M1.7 (LOUT)
- net ROUT is gone; now on net +1V0: RDA58007M1.8 (ROUT)
- net GND: now also U2.57 (GND)
- net GP2 renamed GPIO2
- net GPIO2: now also U2.4 (GPIO2)
- net GP26 renamed GPIO26
- net GPIO26: now also U2.38 (GPIO26_ADC0)
- net GP27 renamed GPIO27
- net GPIO27: now also U2.39 (GPIO27_ADC1)
- net GP3 renamed GPIO3
- net GPIO3: now also U2.5 (GPIO3)
- net GP4 renamed GPIO4
- net GPIO4: now also U2.6 (GPIO4)
- net GP5 renamed GPIO5
- net GPIO5: now also U2.7 (GPIO5)
- net GP6 renamed GPIO6
- net GPIO6: now also U2.8 (GPIO6)
- new net: U2.1 (IOVDD), U2.10 (IOVDD), U2.22 (IOVDD), U2.33 (IOVDD), U2.42 (IOVDD), U2.49 (IOVDD)
- new net: U2.23 (DVDD), U2.50 (DVDD)
- no-connect marks 3 -> 46
