File: project/clockradio/amplifier.kicad_sch (KiCad schematic)
At the start: 7 parts, among them U1 LM386

Commit message: Save experiments.  Save actual project code under code
Connections:
- net +1V0 renamed IN
- net +3.3V renamed VCC
Changed lines of the file:
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@@
-					(unit 1)
-				)
-				(path "/26cce7b5-0449-425b-905b-3af383c44d12/5b629551-fad5-4a3c-ab87-1016e0378cd1"
-					(reference "#PWR07")
 					(unit 1)
 				)
@@
 					(unit 1)
 				)
-				(path "/26cce7b5-0449-425b-905b-3af383c44d12/5b629551-fad5-4a3c-ab87-1016e0378cd1"
-					(reference "C3")
-					(unit 1)
-				)
-			)
-		)
-	)
-	(symbol
-		(lib_id "power:+3.3V")
-		(at 134.62 72.39 0)
-		(unit 1)
-		(exclude_from_sim no)
-		(in_bom yes)
-		(on_board yes)
-		(dnp no)
-		(fields_autoplaced yes)
-		(property "Reference" "#PWR06"
-			(at 134.62 76.2 0)
-			(effects
-				(font
-					(size 1.27 1.27)
-				)
-				(hide yes)
-			)
-		)
-		(property "Value" "+3.3V"
-			(at 134.62 67.31 0)
-			(effects
-				(font
-					(size 1.27 1.27)
-				)
-			)
-		)
-		(property "Footprint" ""
-			(at 134.62 72.39 0)
-			(effects
-				(font
-					(size 1.27 1.27)
-				)
-				(hide yes)
-			)
-		)
-		(property "Datasheet" ""
-			(at 134.62 72.39 0)
-			(effects
-				(font
-					(size 1.27 1.27)
-				)
-				(hide yes)
-			)
-		)
-		(property "Description" "Power symbol creates a global label with name \"+3.3V\""
-			(at 134.62 72.39 0)
-			(effects
-				(font
-					(size 1.27 1.27)
-				)
-				(hide yes)
-			)
-		)
-		(pin "1"
-		)
-		(instances
-			(project ""
-				(path "/26cce7b5-0449-425b-905b-3af383c44d12/0887f379-3559-4bf0-a3a2-19644d2d196f"
-					(reference "#PWR013")
-					(unit 1)
-				)
-				(path "/26cce7b5-0449-425b-905b-3af383c44d12/5b629551-fad5-4a3c-ab87-1016e0378cd1"
-					(reference "#PWR06")
-					(unit 1)
-				)
 			)
 		)
@@
 					(unit 1)
 				)
-				(path "/26cce7b5-0449-425b-905b-3af383c44d12/5b629551-fad5-4a3c-ab87-1016e0378cd1"
-					(reference "R1")
-					(unit 1)
-				)
 			)
 		)
@@
 					(unit 1)
 				)
-				(path "/26cce7b5-0449-425b-905b-3af383c44d12/5b629551-fad5-4a3c-ab87-1016e0378cd1"
-					(reference "LS1")
-					(unit 1)
-				)
 			)
 		)
@@
 					(unit 1)
 				)
-				(path "/26cce7b5-0449-425b-905b-3af383c44d12/5b629551-fad5-4a3c-ab87-1016e0378cd1"
-					(reference "C4")
-					(unit 1)
-				)
 			)
 		)
@@
 					(unit 1)
 				)
-				(path "/26cce7b5-0449-425b-905b-3af383c44d12/5b629551-fad5-4a3c-ab87-1016e0378cd1"
-					(reference "C1")
-					(unit 1)
-				)
 			)
 		)
@@
 					(unit 1)
 				)
-				(path "/26cce7b5-0449-425b-905b-3af383c44d12/5b629551-fad5-4a3c-ab87-1016e0378cd1"
-					(reference "C2")
-					(unit 1)
-				)
-			)
-		)
-	)
-	(symbol
-		(lib_id "power:+1V0")
-		(at 100.33 85.09 0)
-		(unit 1)
-		(exclude_from_sim no)
-		(in_bom yes)
-		(on_board yes)
-		(dnp no)
-		(fields_autoplaced yes)
-		(property "Reference" "#PWR05"
-			(at 100.33 88.9 0)
-			(effects
-				(font
-					(size 1.27 1.27)
-				)
-				(hide yes)
-			)
-		)
-		(property "Value" "+1V0"
-			(at 100.33 80.01 0)
-			(effects
-				(font
-					(size 1.27 1.27)
-				)
-			)
-		)
-		(property "Footprint" ""
-			(at 100.33 85.09 0)
-			(effects
-				(font
-					(size 1.27 1.27)
-				)
-				(hide yes)
-			)
-		)
-		(property "Datasheet" ""
-			(at 100.33 85.09 0)
-			(effects
-				(font
-					(size 1.27 1.27)
-				)
-				(hide yes)
-			)
-		)
-		(property "Description" "Power symbol creates a global label with name \"+1V0\""
-			(at 100.33 85.09 0)
-			(effects
-				(font
-					(size 1.27 1.27)
-				)
-				(hide yes)
-			)
-		)
-		(pin "1"
-		)
-		(instances
-			(project "clockradio"
-				(path "/26cce7b5-0449-425b-905b-3af383c44d12/0887f379-3559-4bf0-a3a2-19644d2d196f"
-					(reference "#PWR012")
-					(unit 1)
-				)
-				(path "/26cce7b5-0449-425b-905b-3af383c44d12/5b629551-fad5-4a3c-ab87-1016e0378cd1"
-					(reference "#PWR05")
-					(unit 1)
-				)
 			)
 		)
@@
 					(unit 1)
 				)
-				(path "/26cce7b5-0449-425b-905b-3af383c44d12/5b629551-fad5-4a3c-ab87-1016e0378cd1"
-					(reference "U1")
-					(unit 1)
-				)
