File: project/clockradio/clockradio.kicad_sch (KiCad schematic)
At the start: 12 parts, among them U1 LM386

Commit message: Updates to project schematic
Parts:
- removed C1: C1 10 µF, symbol Device:C_Polarized
- removed C2: C_Polarized, symbol Device:C_Polarized
- removed C3: 1000µF above 20 Hz, symbol Device:C_Polarized
- removed C4: 0.82 µF above 20 kHz, symbol Device:C
- removed LS1: 8Ω Speaker, symbol Device:Speaker
- removed R1: R 10Ω, symbol Device:R
- removed U1: LM386, symbol Amplifier_Audio:LM386
- added D1: LED, symbol Device:LED
- added R2: R, symbol Device:R
- added SW1: RotaryEncoder_Switch, symbol Device:RotaryEncoder_Switch
- added U2: RP2040, Package_DFN_QFN:QFN-56-1EP_7x7mm_P0.4mm_EP3.2x3.2mm, symbol MCU_RaspberryPi:RP2040
Connections:
- net +3.3V: now also D1.2 (A), SW1.S2, U2.45 (VREG_VOUT)
- net GND: now also R2.2, SW1.C, U2.57 (GND)
- net GP2 renamed GPIO2
- net GPIO2: now also U2.4 (GPIO2)
- net GP26 renamed GPIO26
- net GPIO26: now also U2.38 (GPIO26_ADC0)
- net GP27 renamed GPIO27
- net GPIO27: now also U2.39 (GPIO27_ADC1)
- net GP3 renamed GPIO3
- net GPIO3: now also U2.5 (GPIO3)
- net GP4 renamed GPIO4
- net GPIO4: now also U2.6 (GPIO4)
- net GP5 renamed GPIO5
- net GPIO5: now also U2.7 (GPIO5)
- net GP6 renamed GPIO6
- net GPIO6: now also U2.8 (GPIO6)
- net LOUT renamed amplifierR/IN
- net ROUT renamed amplifierL/IN
- new net: D1.1 (K), R2.1
- new net: U2.1 (IOVDD), U2.10 (IOVDD), U2.22 (IOVDD), U2.33 (IOVDD), U2.42 (IOVDD), U2.49 (IOVDD)
- new net: U2.23 (DVDD), U2.50 (DVDD)
- new net +5V: U2.48 (USB_VDD)
- new net GPIO18: SW1.A, U2.29 (GPIO18)
- new net GPIO19: SW1.B, U2.30 (GPIO19)
- new net GPIO20: SW1.S1, U2.31 (GPIO20)
- no-connect marks 3 -> 38
Other:
- added sheet amplifierL (amplifier.kicad_sch)
- added sheet amplifierR (amplifier.kicad_sch)

Commit message: Save experiments.  Save actual project code under code
Connections:
- net +3.3V: now also SW1.C; no longer SW1.S2
- net GND: now also SW1.S2; no longer SW1.C
- net amplifierL/IN: no longer names the net of RDA58007M1.8 (ROUT)
Other:
- removed sheet amplifierL
