File: project/clockradio_backup/amplifier.kicad_sch (KiCad schematic)
At the start: 7 parts, among them U1 LM386

Commit message: kicad updates
Parts:
- R3: renamed from R1; footprint (none) -> Resistor_THT:R_Axial_DIN0309_L9.0mm_D3.2mm_P12.70mm_Horizontal
- U3: renamed from U1; footprint (none) -> ECE:DIP08
- renumbered C1 to C5, C2 to C6, C3 to C7, C4 to C8, LS1 to LS2
Changed lines of the file:
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@@
 	(hierarchical_label "GND"
 		(shape input)
-		(at 190.5 102.87 270)
+		(at 196.85 99.06 0)
 		(fields_autoplaced yes)
 		(effects
@@
 				(size 1.27 1.27)
 			)
-			(justify right)
+			(justify left)
 		)
 	)
@@
 		(dnp no)
 		(fields_autoplaced yes)
-		(property "Reference" "#PWR07"
+		(property "Reference" "#PWR014"
 			(at 196.85 109.22 0)
 			(effects
@@
 					(unit 1)
 				)
+				(path "/26cce7b5-0449-425b-905b-3af383c44d12/487c280c-3f8d-4ad3-803c-ea9a94b0d6a2"
+					(reference "#PWR01")
+					(unit 1)
+				)
 			)
 		)
@@
 		(dnp no)
 		(fields_autoplaced yes)
-		(property "Reference" "C3"
+		(property "Reference" "C7"
 			(at 172.72 90.1699 0)
 			(effects
@@
 					(unit 1)
 				)
+				(path "/26cce7b5-0449-425b-905b-3af383c44d12/487c280c-3f8d-4ad3-803c-ea9a94b0d6a2"
+					(reference "C3")
+					(unit 1)
+				)
 			)
 		)
@@
 		(dnp no)
 		(fields_autoplaced yes)
-		(property "Reference" "R1"
+		(property "Reference" "R3"
 			(at 171.45 97.7899 0)
 			(effects
@@
 			)
 		)
-		(property "Footprint" ""
+		(property "Footprint" "Resistor_THT:R_Axial_DIN0309_L9.0mm_D3.2mm_P12.70mm_Horizontal"
 			(at 167.132 99.06 90)
 			(effects
@@
 					(unit 1)
 				)
+				(path "/26cce7b5-0449-425b-905b-3af383c44d12/487c280c-3f8d-4ad3-803c-ea9a94b0d6a2"
+					(reference "R1")
+					(unit 1)
+				)
 			)
 		)
@@
 		(dnp no)
 		(fields_autoplaced yes)
-		(property "Reference" "LS1"
+		(property "Reference" "LS2"
 			(at 207.01 87.6299 0)
 			(effects
@@
 					(unit 1)
 				)
+				(path "/26cce7b5-0449-425b-905b-3af383c44d12/487c280c-3f8d-4ad3-803c-ea9a94b0d6a2"
+					(reference "LS1")
+					(unit 1)
+				)
 			)
 		)
@@
 		(dnp no)
 		(fields_autoplaced yes)
-		(property "Reference" "C4"
+		(property "Reference" "C8"
 			(at 175.641 80.01 90)
 			(effects
@@
 					(unit 1)
 				)
+				(path "/26cce7b5-0449-425b-905b-3af383c44d12/487c280c-3f8d-4ad3-803c-ea9a94b0d6a2"
+					(reference "C4")
+					(unit 1)
+				)
 			)
 		)
@@
 		(dnp no)
 		(fields_autoplaced yes)
-		(property "Reference" "C1"
+		(property "Reference" "C5"
 			(at 115.951 77.47 90)
 			(effects
@@
 					(unit 1)
 				)
+				(path "/26cce7b5-0449-425b-905b-3af383c44d12/487c280c-3f8d-4ad3-803c-ea9a94b0d6a2"
+					(reference "C1")
+					(unit 1)
+				)
 			)
 		)
@@
 		(dnp no)
 		(fields_autoplaced yes)
-		(property "Reference" "C2"
+		(property "Reference" "C6"
 			(at 154.94 79.1209 0)
 			(effects
@@
 					(unit 1)
 				)
+				(path "/26cce7b5-0449-425b-905b-3af383c44d12/487c280c-3f8d-4ad3-803c-ea9a94b0d6a2"
+					(reference "C2")
+					(unit 1)
+				)
 			)
 		)
@@
 		(dnp no)
 		(fields_autoplaced yes)
-		(property "Reference" "U1"
+		(property "Reference" "U3"
 			(at 147.32 81.3114 0)
 			(effects
@@
 			)
 		)
-		(property "Footprint" ""
+		(property "Footprint" "ECE:DIP08"
 			(at 139.7 85.09 0)
 			(effects
@@
 					(unit 1)
 				)
+				(path "/26cce7b5-0449-425b-905b-3af383c44d12/487c280c-3f8d-4ad3-803c-ea9a94b0d6a2"
+					(reference "U2")
+					(unit 1)
+				)
