File: project/clockradio_kicad/clockradio.kicad_sch (KiCad schematic)
At the start: 19 parts, among them SW1 RotaryEncoder_Switch, U1 RPi_Pico_TH, U4 LM386

Commit message: Complete project
Parts:
- added DISP2: OLED Display, ECE:OLED_Display_1.3, symbol ECE:OLED Display
- added RTC_I2C_Module_DS1307: ~, symbol Tiny_RTC_DS1307_24C32:RTC_DS1307
Connections:
- net +3.3V: now also DISP2.2 (VDD)
- net GND: now also DISP2.1 (VSS/GND), RTC_I2C_Module_DS1307.2 (GND)
- net GPIO10: now also DISP2.3 (SCLK)
- net GPIO11: now also DISP2.4 (SDA)
- net GPIO12: now also DISP2.6 (DC)
- net GPIO13: now also DISP2.7 (CS)
- net GPIO28: now also RTC_I2C_Module_DS1307.1 (BAT)
- new net GP1014: DISP2.5 (RES)
- new net GPIO16: RTC_I2C_Module_DS1307.4 (SDA)
- new net GPIO17: RTC_I2C_Module_DS1307.5 (SCL)
- no-connect marks 24 -> 32
